File: cheap-wled-controller/cheap-wled-controller.kicad_sch (KiCad schematic)
At the start: 47 parts, among them J10 Conn_01x05_Pin, J2 USB_C_Receptacle, J4 Conn_02x05_Odd_Even, J6 Conn_01x05_Pin, J7 Conn_01x02_Pin, J8 Conn_01x07_Pin, Q3 NMOS, SW1 SW_Push, U1 USBLC6-2SC6, U2 ESP32-S3-WROOM-1-N16R2, U3 CH224K, U4 MX5014S, U7 TPS54202DDC, U9 AMS1117-3.3

Commit message: esp32 s3
Parts:
- added C7, C9: 10u, cheap-wled-controller:C0805, symbol easyeda:CL21A106KOQNNNE
- added C8: 0.1u, cheap-wled-controller:C0805, symbol easyeda:C0805B104K500NT
- added R6, R7: 4k, cheap-wled-controller:R0805, symbol easyeda:ARG05FTC4001N
- added SW2: SW_Push, YULC:SW-SMD_TSA245G00D-250, symbol Switch:SW_Push
- added U5: ESP32-S3-WROOM-1-N4R2, cheap-wled-controller:WIRELM-SMD_ESP32-S3-WROOM-1, symbol easyeda:ESP32-S3-WROOM-1-N4R2
- F2: footprint YULC:FUSE-TH_XF-508P-A-B -> cheap-wled-controller:FUSE-TH_XF-508P-A-B
Connections:
- net +3.3V: now also C8.2, C9.2, R6.1, R7.1, U5.2 (3V3)
- net D+_OUT: now also U5.14 (IO20)
- net D-_OUT: now also U5.13 (IO19)
- net GND: now also C7.1, C8.1, C9.1, SW2.1, U5.1 (GND)
- net GPIO12: now also U5.12 (IO8)
- net GPIO18: now also U5.11 (IO18)
- net GPIO35: now also U5.28 (IO35)
- net GPIO36: now also U5.29 (IO36)
- net GPIO37: now also U5.30 (IO37)
- net GPIO38: now also U5.31 (IO38)
- net GPIO39: now also U5.32 (IO39)
- net GPIO4: now also U5.4 (IO4)
- net GPIO40: now also U5.33 (IO40)
- net GPIO41: now also U5.34 (IO41)
- net GPIO42: now also U5.35 (IO42)
- net GPIO5: now also U5.5 (IO5)
- net GPIO6: now also U5.6 (IO6)
- net LED_DATA: now also U5.39 (IO1)
- net MOS_1: now also U5.24 (IO47)
- net RX: now also U5.36 (RXD0)
- net TX: now also U5.37 (TXD0)
- net VOLT_OUT: now also U5.7 (IO7)
- net MOS_2: no longer names the net of U2.23 (IO21)
- new net: C7.2, R6.2, U5.3 (EN)
- new net: R7.2, SW2.2, U5.27 (IO0)

Commit message: all footprints added
Parts:
- removed C3: 0.1u, cheap-wled-controller:C0805, symbol easyeda:C0805B104K500NT
- removed C4, C6: 10u, cheap-wled-controller:C0805, symbol easyeda:CL21A106KOQNNNE
- removed R1, R9: 4k, cheap-wled-controller:R0805, symbol easyeda:ARG05FTC4001N
- removed SW1: SW_Push, YULC:SW-SMD_TSA245G00D-250, symbol Switch:SW_Push
- removed U2: ESP32-S3-WROOM-1-N16R2, YULC:XCVR_ESP32-S3-WROOM-1-N16R2, symbol ESP32-S3-WROOM-1-N16R2:ESP32-S3-WROOM-1-N16R2
- H1, H2, H3: value MountingHole -> ~; footprint (none) -> MountingHole:MountingHole_3.2mm_M3
- J10: footprint YULC:CONN-TH_5P-P3.81_KF124-3.81-5P -> cheap-wled-controller:CONN-TH_5P-P3.81_KF124-3.81-5P
- J2: footprint Connector_USB:USB_C_Receptacle_G-Switch_GT-USB-7010ASV -> cheap-wled-controller:USB-C_SMD-TYPE-C-31-M-12
- Q3: footprint YULC:DFN-8_L5.9-W5.2-P1.27-LS6.2-BL -> cheap-wled-controller:DFN-8_L5.9-W5.2-P1.27-LS6.2-BL
- SW1: renamed from SW2; footprint YULC:SW-SMD_TSA245G00D-250 -> cheap-wled-controller:SW-SMD_TSA245G00D-250
- U3: footprint ch224k:ESSOP-10_L4.9-W3.9-P1.0-LS6.0-TL-EP -> cheap-wled-controller:ESSOP-10_L4.9-W3.9-P1.0-LS6.0-TL-EP
- U4: footprint YULC:SOIC-8_L4.9-W3.9-P1.27-LS6.0-BL -> cheap-wled-controller:SOIC-8_L4.9-W3.9-P1.27-LS6.0-BL
- renumbered C8 to C3, C9 to C6
Connections:
- net GND: now also U5.40 (GND); no longer U5.1 (GND)
- no-connect marks 33 -> 21
Other:
- moved on the sheet: C29, C3, C30, C6, D2, J10, J6, J7, J8, L2, Q3, R13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

Commit message: leds added
Parts:
- D2, D4: footprint LED_SMD:LED_0603_1608Metric -> cheap-wled-controller:LED0805-R-RD
Changed lines of the file:
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@@
 			)
 		)
-		(property "Footprint" "LED_SMD:LED_0603_1608Metric"
+		(property "Footprint" "cheap-wled-controller:LED0805-R-RD"
 			(at 121.92 100.33 90)
 			(effects
@@
 			)
 		)
-		(property "Footprint" "LED_SMD:LED_0603_1608Metric"
+		(property "Footprint" "cheap-wled-controller:LED0805-R-RD"
 			(at 271.78 85.09 90)
 			(effects
